File: car-bluetooth/car-bluetooth.kicad_pcb (KiCad board)
At the start: 2 copper layers, 99.8 x 48.3 mm, 59 parts, among them J1 EXT, J2 LINE, J3 PWR_1, J4 TAPE_CONTROL, J5 PWR_2, SW1 TAPE_SW, SW2 PLAY/PAUSE, SW3 NEXT/UP, SW4 PREV/DOWN, U1 TLP785, U2 Opamp_Dual_Generic, U5 TLP785, U6 TLP785, U7 buck-converter-3A, U8 Bluetooth-M18

Commit message: sync
Parts:
- removed R16, R17: 4K7, Resistor_SMD:R_0805_2012Metric_Pad1.15x1.40mm_HandSolder
- removed the REF** at (68.1, 141.2)
- removed the REF** at (112.8, 141.2)
- removed the REF** at (129.5, 141.2)
- removed the REF** at (150.1, 141.2)
- removed U5, U6: TLP785, Package_DIP:DIP-4_W10.16mm
- removed U7: buck-converter-3A, custom-footprints:Buck-converter-3A
- added G***: nezumi_logo_3k, custom-footprints:nezumi_logo_3k, F.Cu at (77.5, 144.5)
- added G***: juice-plus_logo_3k, custom-footprints:juice-plus_logo_3k, F.Cu at (76.5, 133.5)
- added J6: MUTE_L, Connector_PinHeader_2.54mm:PinHeader_1x02_P2.54mm_Vertical, F.Cu at (133.5, 113.0)
- added J7: MUTE_R, Connector_PinHeader_2.54mm:PinHeader_1x02_P2.54mm_Vertical, F.Cu at (141.5, 113.0)
- added REF**: MountingHole_3.2mm_M3_DIN965_Pad, MountingHole:MountingHole_3.2mm_M3_DIN965_Pad, F.Cu at (67.5, 141.0)
- added REF**: MountingHole_3.2mm_M3_DIN965_Pad, MountingHole:MountingHole_3.2mm_M3_DIN965_Pad, F.Cu at (117.5, 141.0)
- added REF**: MountingHole_3.2mm_M3_DIN965_Pad, MountingHole:MountingHole_3.2mm_M3_DIN965_Pad, F.Cu at (134.0, 141.0)
- added REF**: MountingHole_3.2mm_M3_DIN965_Pad, MountingHole:MountingHole_3.2mm_M3_DIN965_Pad, F.Cu at (154.5, 141.0)
- added REF**: MountingHole_3.2mm_M3_DIN965_Pad, MountingHole:MountingHole_3.2mm_M3_DIN965_Pad, F.Cu at (120.0, 111.0)
- added U3: OKI-78SR-5/1.5-W36H-C, custom-footprints:OKI-buck-converter-TO220, F.Cu at (93.5, 119.0)
- C1: value 470u -> 330u; footprint Capacitor_THT:CP_Radial_D16.0mm_P7.50mm -> Capacitor_THT:CP_Radial_D10.0mm_P5.00mm
- C14: value 220u -> 330u; footprint Capacitor_THT:CP_Radial_D12.5mm_P5.00mm -> Capacitor_THT:CP_Radial_D10.0mm_P5.00mm
- C16, C7: value 100u -> 330u; footprint Capacitor_THT:CP_Radial_D12.5mm_P5.00mm -> Capacitor_THT:CP_Radial_D10.0mm_P5.00mm
- J4: footprint Connector_JST:JST_XH_B05B-XH-A_1x05_P2.50mm_Vertical -> Connector_JST:JST_XH_B03B-XH-A_1x03_P2.50mm_Vertical
- R22: value 2K2 -> 4K7
- U1: footprint Package_DIP:DIP-4_W10.16mm -> Package_DIP:DIP-4_W7.62mm_Socket
- moved R22 41.9 mm to (96.7, 150.2), turned to 0 degrees
- moved D2 36.3 mm to (92.0, 150.2), turned to 180 degrees
- moved C14 34.2 mm to (76.5, 110.5)
- moved C1 32.3 mm to (109.5, 110.2), turned to 180 degrees
- moved C7 22.5 mm to (98.5, 110.2), turned to 180 degrees
- moved R4 20.8 mm to (121.0, 120.8)
- moved R8 20.8 mm to (109.5, 117.5), turned to 270 degrees
- moved C16 20.2 mm to (87.5, 110.5), turned to 180 degrees
- moved C10 19.1 mm to (115.0, 117.5), turned to 90 degrees
- moved R7 18.1 mm to (130.0, 128.2)
- moved U1 18.1 mm to (76.2, 119.8), turned to 270 degrees
- moved R9 15.9 mm to (112.2, 117.5)
- moved R2 14.5 mm to (148.0, 113.0), turned to 180 degrees
- moved C6 13.2 mm to (100.0, 120.0), turned to 270 degrees
- moved C2 11.6 mm to (104.0, 124.5), turned to 0 degrees
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Connections:
- C16 pad 1: 12V -> MOTOR
- C6 pad 1: 12V -> MOTOR
- J4 pad 1: MOTOR -> TAPE
- J4 pad 2: Net-(J4-Pad2) -> COM
- J4 pad 3: TAPE -> MOTOR
Routing:
- net MOTOR: track 86.0 -> 139.0 mm
- net Net-(C5-Pad2): track 36.3 -> 9.42 mm, vias 1 -> 0
- net Net-(C8-Pad2): track 28.4 -> 10.3 mm
- net Net-(R17-Pad2): track 13.4 -> 0.00 mm
- net EXT_R: track 14.9 -> 27.7 mm
- net BLUETOOTH_L: track 7.79 -> 17.2 mm
- net Net-(C3-Pad2): track 5.82 -> 14.9 mm
- net Net-(C2-Pad2): track 5.81 -> 14.0 mm
- net V_BIAS: track 31.3 -> 39.1 mm
- net 5V_EN: track 6.98 -> 0.00 mm
- net Net-(R18-Pad1): track 59.4 -> 65.5 mm
- net Net-(R3-Pad1): track 9.06 -> 3.22 mm
- net Net-(R16-Pad1): track 5.47 -> 0.00 mm
- net Net-(C12-Pad1): track 38.7 -> 33.4 mm
- net 12V: track 91.5 -> 87.7 mm
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Other:
- board text added: "Chip@ SnakeOilDev.com"
- board text added: "For MB942709 RX-277"
- board text added: "GND VCC"
- board text added: "LIN_R LIN_L"
- board text added: "MOT A_L A_R MUT GND VCC"
- board text added: "MUTE_EXT"
- board text added: "Rev.3"
- board text added: "TAPE COM MOT"
- board text added: "VCC GND MUT"
- board text removed: "ChipCE"
- board text removed: "For MB942709"
- board text removed: "RX-277 cassette deck"
- board text removed: "Rev.1"
- board text removed: "SnakeOilDev"
