File: car-bluetooth/car-bluetooth.sch (KiCad schematic (older format))
At the start: 55 parts, among them J1 EXT, J2 LINE, J3 PWR_1, J4 TAPE_CONTROL, J5 PWR_2, SW1 TAPE_SW, SW2 PLAY/PAUSE, SW3 NEXT/UP, SW4 PREV/DOWN, U1 TLP785, U2 Opamp_Dual_Generic, U5 TLP785, U6 TLP785, U7 buck-converter-3A, U8 Bluetooth-M18

Commit message: sync
Parts:
- removed J4: TAPE_CONTROL, Connector_JST:JST_XH_B05B-XH-A_1x05_P2.50mm_Vertical, symbol Connector:Conn_01x05_Female
- removed R16, R17: 4K7, Resistor_SMD:R_0805_2012Metric_Pad1.15x1.40mm_HandSolder, symbol Device:R_US
- removed U5, U6: TLP785, Package_DIP:DIP-4_W10.16mm, symbol dk_Optoisolators-Transistor-Photovoltaic-Output:LTV-356T
- removed U7: buck-converter-3A, custom-footprints:Buck-converter-3A, symbol custom-symbols:buck-converter-3A
- added J4: TAPE_CONTROL, Connector_JST:JST_XH_B03B-XH-A_1x03_P2.50mm_Vertical, symbol Connector:Conn_01x03_Female
- added J6: MUTE_L, Connector_PinHeader_2.54mm:PinHeader_1x02_P2.54mm_Vertical, symbol Connector:Conn_01x02_Male
- added J7: MUTE_R, Connector_PinHeader_2.54mm:PinHeader_1x02_P2.54mm_Vertical, symbol Connector:Conn_01x02_Male
- added U3: OKI-78SR-5/1.5-W36H-C, custom-footprints:OKI-buck-converter-TO220, symbol dk_PMIC-Voltage-Regulators-Linear:L7805CV
- C1: value 470u -> 330u; footprint Capacitor_THT:CP_Radial_D16.0mm_P7.50mm -> Capacitor_THT:CP_Radial_D10.0mm_P5.00mm
- C14: value 220u -> 330u; footprint Capacitor_THT:CP_Radial_D12.5mm_P5.00mm -> Capacitor_THT:CP_Radial_D10.0mm_P5.00mm
- C16, C7: value 100u -> 330u; footprint Capacitor_THT:CP_Radial_D12.5mm_P5.00mm -> Capacitor_THT:CP_Radial_D10.0mm_P5.00mm
- R22: value 2K2 -> 4K7
- U1: footprint Package_DIP:DIP-4_W10.16mm -> Package_DIP:DIP-4_W7.62mm_Socket
Connections:
- net 12V: no longer C16.1, C6.1
- net 5V: now also U3.3 (OUT)
- net COM: now also J4.2 (Pin_2)
- net EXT_L: now also J6.2 (Pin_2)
- net EXT_R: now also J7.2 (Pin_2)
- net GND: now also J6.1 (Pin_1), J7.1 (Pin_1), U3.2 (GND)
- net MOTOR: now also C16.1, C6.1, J4.3 (Pin_3), U3.1 (IN)
- net TAPE: now also J4.1 (Pin_1)
- no-connect marks 3 -> 2
Other:
- moved on the sheet: C1, C14, C15, C6, D2, R22, R3, SW1, U1
