File: direct-pt1000-stick/direct-pt1000-stick.kicad_pcb (KiCad board)
At the start: 2 copper layers, 18 x 60 mm, 13 parts, among them J1 BRIDGE/a, J10 M3_hole, J2 BRIDGE/b, J3 C_TH_1/a, J4 C_TH_1/a, J5 C_TH_2/a, J6 C_TH_2/a, J7 C_TH_3/a, J8 C_TH_3/a, J9 M3_hole

Commit message: sync
Parts:
- removed J10, J9: M3_hole, MountingHole:MountingHole_3.2mm_M3_DIN965_Pad
- removed J3, J4: C_TH_1/a, Connector_JST:JST_XH_B2B-XH-A_1x02_P2.50mm_Vertical
- removed J5, J6: C_TH_2/a, Connector_JST:JST_XH_B2B-XH-A_1x02_P2.50mm_Vertical
- removed J7, J8: C_TH_3/a, Connector_JST:JST_XH_B2B-XH-A_1x02_P2.50mm_Vertical
- removed R2, R3: 1K5, Resistor_SMD:R_0805_2012Metric
- added U1: BTT_OCTOPUS_WIFI_SLOT, custom-footprints:BTT_OCTOPUS_WIFI_SLOT, F.Cu at (143.6, 94.6)
- J1: value BRIDGE/a -> PT1000_P1/a; footprint Connector_JST:JST_XH_B3B-XH-A_1x03_P2.50mm_Vertical -> Connector_JST:JST_XH_S2B-XH-A-1_1x02_P2.50mm_Horizontal; moved to B.Cu
- J2: value BRIDGE/b -> PT1000_P1/b; footprint Connector_JST:JST_XH_B3B-XH-A_1x03_P2.50mm_Vertical -> Connector_JST:JST_XH_S2B-XH-A-1_1x02_P2.50mm_Horizontal; moved to B.Cu
- R1: footprint Resistor_SMD:R_0805_2012Metric -> Resistor_SMD:R_0805_2012Metric_Pad1.20x1.40mm_HandSolder
- moved J1 49.3 mm to (134.9, 102.0)
- moved J2 36.1 mm to (143.4, 102.0)
- moved R1 33.4 mm to (134.9, 112.4), turned to 0 degrees
Connections:
- net IO renamed Net-(J1-Pad1)
- J1 pad 2: GND -> Net-(J1-Pad2)
- J2 pad 2: GND -> Net-(J1-Pad2)
- R1 pad 1: 3.3V -> 3V3
- R1 pad 2: Net-(J3-Pad2) -> Net-(J1-Pad2)
Routing:
- net 3.3V: track 46.7 -> 0.00 mm, vias 3 -> 0
- net Net-(J1-Pad1): track 37.4 -> 9.88 mm
- net Net-(J1-Pad2): track 0.00 -> 20.3 mm
- net Net-(J7-Pad2): track 11.0 -> 0.00 mm
- net Net-(J5-Pad2): track 11.0 -> 0.00 mm
- net Net-(J3-Pad2): track 11.0 -> 0.00 mm
- net 3V3: track 0.00 -> 3.02 mm
- removed copper zone on B.Cu, net GND
- removed copper zone on F.Cu, net GND
Other:
- board size 18 x 60 mm -> 21.6 x 20.3 mm
- board text added: "<<config>> pullup_resistor : 1000"
- board text added: "Bottom side"
- board text added: "Direct PT1000 Stick"
- board text added: "GND"
- board text added: "PT1000"
- board text added: "TEMP"
- board text removed: "DIRECT PT1000 STICK"
- board text removed: "GND T1"
- board text removed: "GND T2"
- board text removed: "GND T3"
- board text removed: "IO GND 3.3V"
- board text removed: "https://github.com/ChipCE/juice-plus-pcb"
