File: direct-pt1000-stick/direct-pt1000-stick.sch (KiCad schematic (older format))
At the start: 13 parts, among them J1 BRIDGE/a, J10 M3_hole, J2 BRIDGE/b, J3 C_TH_1/a, J4 C_TH_1/a, J5 C_TH_2/a, J6 C_TH_2/a, J7 C_TH_3/a, J8 C_TH_3/a, J9 M3_hole

Commit message: sync
Parts:
- removed J1: BRIDGE/a, Connector_JST:JST_XH_B3B-XH-A_1x03_P2.50mm_Vertical, symbol Connector:Conn_01x03_Female
- removed J10, J9: M3_hole, MountingHole:MountingHole_3.2mm_M3_DIN965_Pad, symbol Connector:Conn_01x01_Female
- removed J2: BRIDGE/b, Connector_JST:JST_XH_B3B-XH-A_1x03_P2.50mm_Vertical, symbol Connector:Conn_01x03_Female
- removed J3, J4: C_TH_1/a, Connector_JST:JST_XH_B2B-XH-A_1x02_P2.50mm_Vertical, symbol Connector:Conn_01x02_Female
- removed J5, J6: C_TH_2/a, Connector_JST:JST_XH_B2B-XH-A_1x02_P2.50mm_Vertical, symbol Connector:Conn_01x02_Female
- removed J7, J8: C_TH_3/a, Connector_JST:JST_XH_B2B-XH-A_1x02_P2.50mm_Vertical, symbol Connector:Conn_01x02_Female
- removed R2, R3: 1K5, Resistor_SMD:R_0805_2012Metric, symbol Device:R_US
- added J1: PT1000_P1/a, Connector_JST:JST_XH_S2B-XH-A-1_1x02_P2.50mm_Horizontal, symbol Connector:Conn_01x02_Female
- added J2: PT1000_P1/b, Connector_JST:JST_XH_S2B-XH-A-1_1x02_P2.50mm_Horizontal, symbol Connector:Conn_01x02_Female
- added U1: BTT_OCTOPUS_WIFI_SLOT, custom-footprints:BTT_OCTOPUS_WIFI_SLOT, symbol custom-symbols:BTT_OCTOPUS_WIFI_SLOT
- R1: footprint Resistor_SMD:R_0805_2012Metric -> Resistor_SMD:R_0805_2012Metric_Pad1.20x1.40mm_HandSolder
Connections:
- net at R1.2: now also J1.2 (Pin_2), J2.2 (Pin_2)
- net 3.3V renamed 3V3
- net 3V3: now also U1.8 (3V3)
- new net: J1.1 (Pin_1), J2.1 (Pin_1)
- no-connect marks 2 -> 15
