File: adapter-board/adapter-board.kicad_pcb (KiCad board)
At the start: 4 copper layers, 80.3 x 25.7 mm, 20 parts, among them J1 TAPE, J2 Conn_01x02_Female, J3 HEADER3, J4 HEADER1, J5 BLU, J6 SOP16, J7 HEADER4, J8 HEADER2, J9 Conn_01x05_Female

Commit message: sync
Parts:
- added C1: C, Capacitor_SMD:C_0805_2012Metric_Pad1.18x1.45mm_HandSolder, F.Cu at (155.4, 73.2)
- added C2: C, Capacitor_SMD:C_0805_2012Metric_Pad1.18x1.45mm_HandSolder, F.Cu at (155.4, 75.9)
- added C3: C, Capacitor_SMD:C_0805_2012Metric_Pad1.18x1.45mm_HandSolder, B.Cu at (156.2, 84.3)
- added C4: C, Capacitor_SMD:C_0805_2012Metric_Pad1.18x1.45mm_HandSolder, B.Cu at (156.2, 86.6)
- added C5: C, Capacitor_SMD:C_0805_2012Metric_Pad1.18x1.45mm_HandSolder, F.Cu at (152.1, 90.7)
- added C6: C, Capacitor_SMD:C_0805_2012Metric_Pad1.18x1.45mm_HandSolder, F.Cu at (130.6, 84.3)
- added C7: C, Capacitor_SMD:C_0805_2012Metric_Pad1.18x1.45mm_HandSolder, F.Cu at (126.5, 84.3)
- added C8: C, Capacitor_SMD:C_0805_2012Metric_Pad1.18x1.45mm_HandSolder, F.Cu at (140.0, 84.3)
- added D3: LED, LED_SMD:LED_0805_2012Metric_Pad1.15x1.40mm_HandSolder, F.Cu at (140.0, 86.6)
- added J10: Conn_01x03_Male, Connector_PinHeader_2.54mm:PinHeader_1x03_P2.54mm_Vertical, F.Cu at (159.8, 90.9)
- added J11: Conn_01x02_Male, Connector_PinHeader_2.54mm:PinHeader_1x02_P2.54mm_Vertical, F.Cu at (159.5, 75.7)
- added J12: Conn_01x02_Male, Connector_PinHeader_2.54mm:PinHeader_1x02_P2.54mm_Vertical, F.Cu at (134.6, 90.2)
- added R3: R_US, Resistor_SMD:R_0805_2012Metric_Pad1.20x1.40mm_HandSolder, F.Cu at (126.5, 86.6)
- added R4: R_US, Resistor_SMD:R_0805_2012Metric_Pad1.20x1.40mm_HandSolder, F.Cu at (135.4, 84.3)
- added Y1: Crystal, Crystal:Crystal_C38-LF_D3.0mm_L8.0mm_Horizontal_1EP_style1, F.Cu at (152.1, 69.8)
- moved J5 4.70 mm to (133.3, 67.8)
- moved J4 2.29 mm to (149.9, 73.2)
- moved J6 2.29 mm to (156.2, 82.7)
- moved J8 2.29 mm to (162.6, 90.9)
Connections:
- J3 pad 1: Net-(J3-Pad1) -> B_GND
- J4 pad 1: Net-(J4-Pad1) -> R_GND
- J4 pad 4: Net-(J4-Pad4) -> R_VCC
- J4 pad 5: Net-(J4-Pad5) -> R_GND
- J4 pad 8: Net-(J4-Pad8) -> R_VCC
- J5 pad 1: Net-(J3-Pad1) -> B_GND
- J5 pad 11: Net-(J5-Pad11) -> B_GND
- J5 pad 16: Net-(J5-Pad16) -> B_VCC
- J5 pad 17: Net-(J5-Pad17) -> B_VCC
- J5 pad 18: Net-(J5-Pad18) -> B_GND
- J5 pad 19: Net-(J5-Pad19) -> B_GND
- J5 pad 20: Net-(J5-Pad20) -> B_GND
- J6 pad 1: Net-(J4-Pad1) -> R_GND
- J6 pad 11: Net-(J6-Pad11) -> R_GND
- J6 pad 12: Net-(J6-Pad12) -> R_GND
- J6 pad 15: Net-(J6-Pad15) -> R_GND
- J6 pad 4: Net-(J4-Pad4) -> R_VCC
- J6 pad 5: Net-(J4-Pad5) -> R_GND
- J6 pad 8: Net-(J4-Pad8) -> R_VCC
- J6 pad 9: Net-(J6-Pad9) -> R_GND
- J7 pad 1: Net-(J5-Pad11) -> B_GND
- J7 pad 10: Net-(J5-Pad20) -> B_GND
- J7 pad 6: Net-(J5-Pad16) -> B_VCC
- J7 pad 7: Net-(J5-Pad17) -> B_VCC
- J7 pad 8: Net-(J5-Pad18) -> B_GND
- J7 pad 9: Net-(J5-Pad19) -> B_GND
- J8 pad 1: Net-(J6-Pad9) -> R_GND
- J8 pad 3: Net-(J6-Pad11) -> R_GND
- J8 pad 4: Net-(J6-Pad12) -> R_GND
- J8 pad 7: Net-(J6-Pad15) -> R_GND
Routing:
- net R_GND: track 0.00 -> 29.8 mm
- net Net-(J3-Pad2): track 5.54 -> 24.5 mm
- net B_VCC: track 0.00 -> 16.3 mm, vias 0 -> 1
- net R_VCC: track 0.00 -> 16.3 mm
- net Net-(C2-Pad1): track 4.10 -> 16.6 mm, vias 0 -> 1
- net Net-(C1-Pad1): track 5.54 -> 17.3 mm, vias 0 -> 1
- net Net-(C6-Pad2): track 0.00 -> 10.4 mm
- net Net-(J3-Pad7): track 4.73 -> 13.8 mm, vias 0 -> 1
- net Net-(C7-Pad1): track 4.30 -> 13.1 mm, vias 0 -> 1
- net Net-(C3-Pad2): track 0.00 -> 7.64 mm, vias 0 -> 1
- net Net-(J5-Pad11): track 6.67 -> 0.00 mm
- net Net-(J4-Pad1): track 6.34 -> 0.00 mm
- net Net-(C4-Pad1): track 3.98 -> 10.0 mm
- net Net-(C3-Pad1): track 3.57 -> 9.54 mm
- net Net-(J5-Pad20): track 5.95 -> 0.00 mm
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- added copper zone on B.Cu, net B_GND
- added copper zone on F.Cu, net B_GND
- added copper zone on B.Cu, net R_GND
- added copper zone on F.Cu, net R_GND
Other:
- board text added: "A"
- board text added: "G"
- board text added: "L"
- board text added: "R"
