File: esp32-button/esp32-button.kicad_pcb (KiCad board)
At the start: 2 copper layers, 22 x 60 mm, 12 parts, among them J3 Conn_01x02_Female, SW1 SW_Push, SW2 SW_Push, SW3 SW_Push, SW4 SW_Push, SW5 SW_Push, SW6 SW_Push, U1 XIAO-ESP32C

Commit message: sync
Parts:
- C1: renamed from C7; moved to B.Cu
- C2: renamed from C8; moved to B.Cu
- D1: moved to B.Cu
- R1: renamed from R13; moved to B.Cu
- moved J3 7.69 mm to (144.0, 89.3)
- moved C2 6.57 mm to (142.5, 99.5)
- moved C1 5.58 mm to (145.5, 99.5)
- moved R1 2.50 mm to (152.5, 75.0)
- moved D1 1.95 mm to (152.5, 70.0)
Connections:
- R1 pad 2: Net-(R13-Pad2) -> Net-(R1-Pad2)
- U1 pad 11: Net-(R13-Pad2) -> Net-(U1-Pad11)
- U1 pad 8: Net-(U1-Pad8) -> Net-(R1-Pad2)
Routing:
- net Net-(R13-Pad2): track 40.8 -> 0.00 mm, vias 1 -> 0
- net Net-(R1-Pad2): track 0.00 -> 28.7 mm
- net 5V: track 39.7 -> 35.4 mm, vias 2 -> 0
- net Net-(SW4-Pad2): track 28.8 -> 30.1 mm
- net Net-(SW5-Pad2): track 36.3 -> 37.5 mm
- net Net-(D1-Pad2): track 2.45 -> 3.00 mm
- net GND: vias 11 -> 12

Commit message: sync
Parts:
- added J1: Conn_01x02_Female, custom-footprints:solder-pad-2p, B.Cu at (144.0, 79.2)
- added J2: Conn_01x02_Female, custom-footprints:solder-pad-2p, B.Cu at (144.0, 68.8)
Routing:
- net 5V: track 35.4 -> 69.7 mm
- net GND: vias 12 -> 10
Other:
- board text added: "5V"
- board text added: "D1"
- board text added: "D2"
- board text added: "D3"
- board text added: "D4"
- board text added: "D5"
- board text added: "D6"
- board text added: "D7"
- board text added: "GND"
- board text added: "Rev.1"
- board text added: "Xiao Mini Button Extender"
