File: esp32-button/esp32-button.sch (KiCad schematic (older format))
At the start: 12 parts, among them J3 Conn_01x02_Female, SW1 SW_Push, SW2 SW_Push, SW3 SW_Push, SW4 SW_Push, SW5 SW_Push, SW6 SW_Push, U1 XIAO-ESP32C

Commit message: sync
Parts:
- renumbered C7 to C1, C8 to C2, R13 to R1
Connections:
- net at U1.11 (D10): no longer R1.2
- net at U1.8 (D7): now also R1.2
Changed lines of the file:
@@
 $EndComp
 $Comp
-L Device:C C7
+L Device:C C1
 U 1 1 6364E16C
 P 5150 1350
-F 0 "C7" H 5265 1396 50  0000 L CNN
+F 0 "C1" H 5265 1396 50  0000 L CNN
 F 1 "1u" H 5265 1305 50  0000 L CNN
 F 2 "Capacitor_SMD:C_0805_2012Metric_Pad1.18x1.45mm_HandSolder" H 5188 1200 50  0001 C CNN
@@
 NoConn ~ 3450 1200
 $Comp
-L Device:C C8
+L Device:C C2
 U 1 1 6374DF10
 P 5500 1350
-F 0 "C8" H 5615 1396 50  0000 L CNN
+F 0 "C2" H 5615 1396 50  0000 L CNN
 F 1 "100n" H 5615 1305 50  0000 L CNN
 F 2 "Capacitor_SMD:C_0805_2012Metric_Pad1.18x1.45mm_HandSolder" H 5538 1200 50  0001 C CNN
@@
 NoConn ~ 4150 1600
 NoConn ~ 4150 1700
-NoConn ~ 4150 1800
-$Comp
-L Device:R_US R13
+NoConn ~ 4150 1500
+$Comp
+L Device:R_US R1
 U 1 1 637A5B15
 P 4600 2050
-F 0 "R13" V 4395 2050 50  0000 C CNN
+F 0 "R1" V 4395 2050 50  0000 C CNN
 F 1 "1K" V 4486 2050 50  0000 C CNN
 F 2 "Resistor_SMD:R_0805_2012Metric_Pad1.20x1.40mm_HandSolder" V 4640 2040 50  0001 C CNN
@@
 $EndComp
 Wire Wire Line
-	4150 1500 4450 1500
-Wire Wire Line
-	4450 1500 4450 2050
-Wire Wire Line
 	4750 2050 4900 2050
 Wire Wire Line
@@
 Connection ~ 2200 2800
 $Comp
-L power:GND #PWR?
+L power:GND #PWR0101
 U 1 1 638A6EF5
 P 2200 3400
-F 0 "#PWR?" H 2200 3150 50  0001 C CNN
+F 0 "#PWR0101" H 2200 3150 50  0001 C CNN
 F 1 "GND" H 2205 3227 50  0000 C CNN
 F 2 "" H 2200 3400 50  0001 C CNN
@@
 Connection ~ 2200 3200
 NoConn ~ 4150 1400
+Wire Wire Line
+	4150 1800 4450 1800
+Wire Wire Line
+	4450 1800 4450 2050
 $EndSCHEMATC

Commit message: sync
Parts:
- added J1, J2: Conn_01x02_Female, custom-footprints:solder-pad-2p, symbol Connector:Conn_01x02_Female
Connections:
- net 5V: now also J1.2 (Pin_2), J2.2 (Pin_2)
- net GND: now also J1.1 (Pin_1), J2.1 (Pin_1)
Changed lines of the file:
@@
 Wire Wire Line
 	4450 1800 4450 2050
+$Comp
+L Connector:Conn_01x02_Female J1
+U 1 1 6369FDD5
+P 6900 2000
+F 0 "J1" H 6792 1675 50  0000 C CNN
+F 1 "Conn_01x02_Female" H 6792 1766 50  0000 C CNN
+F 2 "custom-footprints:solder-pad-2p" H 6900 2000 50  0001 C CNN
+F 3 "~" H 6900 2000 50  0001 C CNN
+	1    6900 2000
+	-1   0    0    1
+$EndComp
+$Comp
+L Connector:Conn_01x02_Female J2
+U 1 1 636A0A9C
+P 6900 2300
+F 0 "J2" H 6792 1975 50  0000 C CNN
+F 1 "Conn_01x02_Female" H 6792 2066 50  0000 C CNN
+F 2 "custom-footprints:solder-pad-2p" H 6900 2300 50  0001 C CNN
+F 3 "~" H 6900 2300 50  0001 C CNN
+	1    6900 2300
+	-1   0    0    1
+$EndComp
+Text GLabel 7350 1900 2    50   Input ~ 0
+5V
+Text GLabel 7350 2000 2    50   Input ~ 0
+GND
+Text GLabel 7350 2200 2    50   Input ~ 0
+5V
+Text GLabel 7350 2300 2    50   Input ~ 0
+GND
+Wire Wire Line
+	7100 1900 7350 1900
+Wire Wire Line
+	7100 2000 7350 2000
+Wire Wire Line
+	7100 2200 7350 2200
+Wire Wire Line
+	7100 2300 7350 2300
 $EndSCHEMATC
