File: fan-expander/fan-expander.kicad_pcb (KiCad board)
At the start: 4 copper layers, 18 parts, among them J1 O1, J10 O5, J11 O6, J2 FAN_PWR, J3 IO, J4 CH_SEL, J5 CH1_SEL, J6 CH2_SEL, J7 O2, J8 O3, J9 O4, U1 4069

Commit message: sync!
Parts:
- removed J10: O5, Connector_JST:JST_XH_B3B-XH-A_1x03_P2.50mm_Vertical
- removed J11: O6, Connector_JST:JST_XH_B3B-XH-A_1x03_P2.50mm_Vertical
- removed J6: CH2_SEL, Connector_PinHeader_2.54mm:PinHeader_1x06_P2.54mm_Vertical
- removed J7: O2, Connector_JST:JST_XH_B3B-XH-A_1x03_P2.50mm_Vertical
- removed J8: O3, Connector_JST:JST_XH_B3B-XH-A_1x03_P2.50mm_Vertical
- removed J9: O4, Connector_JST:JST_XH_B3B-XH-A_1x03_P2.50mm_Vertical
- removed JP1, JP2: Jumper_NC_Small, Connector_PinHeader_2.54mm:PinHeader_1x02_P2.54mm_Vertical
- removed U1: 4069, Package_DIP:DIP-14_W7.62mm
- added D1: LED, LED_SMD:LED_0805_2012Metric_Pad1.15x1.40mm_HandSolder, F.Cu at (155.5, 70.5)
- added D2: LED, LED_SMD:LED_0805_2012Metric_Pad1.15x1.40mm_HandSolder, F.Cu at (151.0, 70.5)
- added R3: R_US, Resistor_SMD:R_0805_2012Metric_Pad1.20x1.40mm_HandSolder, F.Cu at (146.5, 88.5)
- added R4: R_US, Resistor_SMD:R_0805_2012Metric_Pad1.20x1.40mm_HandSolder, F.Cu at (151.0, 75.0)
- J1: value O1 -> FAN_PWR; footprint Connector_JST:JST_XH_B3B-XH-A_1x03_P2.50mm_Vertical -> Connector_JST:JST_XH_B2B-XH-A_1x02_P2.50mm_Vertical
- J2: value FAN_PWR -> Conn_01x03_Female; footprint Connector_JST:JST_VH_B2P-VH-FB-B_1x02_P3.96mm_Vertical -> Connector_JST:JST_XH_B3B-XH-A_1x03_P2.50mm_Vertical
- J3: value IO -> FAN_OUTPUT_1
- J4: value CH_SEL -> FAN_OUTPUT_2; footprint Connector_PinHeader_2.54mm:PinHeader_1x06_P2.54mm_Vertical -> Connector_JST:JST_XH_B4B-XH-A_1x04_P2.50mm_Vertical
- J5: value CH1_SEL -> Conn_02x03_Odd_Even; footprint Connector_PinHeader_2.54mm:PinHeader_1x06_P2.54mm_Vertical -> Connector_PinHeader_2.54mm:PinHeader_2x03_P2.54mm_Vertical
- moved J1 42.1 mm to (156.0, 96.0), turned to 270 degrees
- moved J4 39.6 mm to (154.5, 57.0), turned to 270 degrees
- moved R1 36.1 mm to (155.5, 75.0), turned to 270 degrees
- moved J3 34.3 mm to (145.5, 64.5), turned to 90 degrees
- moved J2 24.0 mm to (149.0, 98.5), turned to 180 degrees
- moved J5 17.8 mm to (155.0, 81.5), turned to 270 degrees
- moved R2 15.5 mm to (144.0, 88.5), turned to 270 degrees
Connections:
- J1 pad 1: F_VCC -> FAN_VCC
- J2 pad 1: F_VCC -> IO_VCC
- J2 pad 2: GND -> TAC
- J3 pad 1: IO_VCC -> FAN_VCC
- J3 pad 2: GND -> PWM
- J3 pad 3: CH1 -> TAC
- J3 pad 4: CH2 -> GND
- J4 pad 1: Net-(J4-Pad1) -> FAN_VCC
- J4 pad 2: Net-(J4-Pad2) -> PWM
- J4 pad 3: Net-(J4-Pad3) -> TAC
- J4 pad 4: Net-(J4-Pad4) -> GND
- J5 pad 1: CH1 -> Net-(J5-Pad1)
- J5 pad 2: CH1 -> Net-(J5-Pad2)
- J5 pad 3: CH1 -> IO_VCC
- J5 pad 4: CH1 -> IO_VCC
- J5 pad 5: CH1 -> Net-(J5-Pad5)
- J5 pad 6: CH1 -> Net-(J5-Pad6)
- R1 pad 1: IO_VCC -> Net-(D1-Pad2)
- R1 pad 2: Net-(JP1-Pad2) -> IO_VCC
- R2 pad 1: IO_VCC -> Net-(J5-Pad5)
- R2 pad 2: Net-(JP2-Pad2) -> PWM
Routing:
- net FAN_VCC: track 0.00 -> 83.7 mm
- net PWM: track 0.00 -> 73.2 mm, vias 0 -> 1
- net TAC: track 0.00 -> 67.2 mm
- net OUT5: track 31.4 -> 0.00 mm
- net OUT3: track 30.7 -> 0.00 mm
- net IO_VCC: track 0.00 -> 30.2 mm
- net OUT4: track 27.0 -> 0.00 mm
- net OUT1: track 26.3 -> 0.00 mm
- net CH1: track 24.3 -> 0.00 mm
- net CH2: track 22.7 -> 0.00 mm
- net Net-(J4-Pad1): track 22.3 -> 0.00 mm
- net OUT2: track 21.0 -> 0.00 mm
- net Net-(J4-Pad6): track 19.8 -> 0.00 mm
- net Net-(J4-Pad2): track 17.3 -> 0.00 mm
- net OUT6: track 15.8 -> 0.00 mm
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- added copper zone on F.Cu, net FAN_VCC
- removed copper zone on F.Cu, net F_VCC
Other:
- board outline added: 18 x 64 mm
- copper layers 4 -> 2
- board text added: "+"
- board text added: "-"
- board text added: "FAN IO"
- board text added: "FAN OUTPUT"
- board text added: "FAN PWR"
- board text added: "Fan Controller"
- board text added: "GND"
- board text added: "IO_VCC"
- board text added: "NC"
- board text added: "P"
- board text added: "PULLUP"
- board text added: "PWM"
- board text added: "PWM_SIG"
- board text added: "Rev.1"
- board text added: "T"
- board text added: "TAC"
- board text added: "TAC_SIG"
- board text added: "VCC"
