File: fan-expander/fan-expander.sch (KiCad schematic (older format))
At the start: 16 parts, among them J1 O1, J10 O5, J11 O6, J2 FAN_PWR, J3 IO, J4 CH_SEL, J5 CH1_SEL, J6 CH2_SEL, J7 O2, J8 O3, J9 O4, U1 4069

Commit message: sync!
Parts:
- removed J1: O1, Connector_JST:JST_XH_B3B-XH-A_1x03_P2.50mm_Vertical, symbol Connector:Conn_01x03_Female
- removed J10: O5, Connector_JST:JST_XH_B3B-XH-A_1x03_P2.50mm_Vertical, symbol Connector:Conn_01x03_Female
- removed J11: O6, Connector_JST:JST_XH_B3B-XH-A_1x03_P2.50mm_Vertical, symbol Connector:Conn_01x03_Female
- removed J2: FAN_PWR, Connector_JST:JST_VH_B2P-VH-FB-B_1x02_P3.96mm_Vertical, symbol Connector:Conn_01x02_Female
- removed J4: CH_SEL, Connector_PinHeader_2.54mm:PinHeader_1x06_P2.54mm_Vertical, symbol Connector:Conn_01x06_Male
- removed J5: CH1_SEL, Connector_PinHeader_2.54mm:PinHeader_1x06_P2.54mm_Vertical, symbol Connector:Conn_01x06_Male
- removed J6: CH2_SEL, Connector_PinHeader_2.54mm:PinHeader_1x06_P2.54mm_Vertical, symbol Connector:Conn_01x06_Male
- removed J7: O2, Connector_JST:JST_XH_B3B-XH-A_1x03_P2.50mm_Vertical, symbol Connector:Conn_01x03_Female
- removed J8: O3, Connector_JST:JST_XH_B3B-XH-A_1x03_P2.50mm_Vertical, symbol Connector:Conn_01x03_Female
- removed J9: O4, Connector_JST:JST_XH_B3B-XH-A_1x03_P2.50mm_Vertical, symbol Connector:Conn_01x03_Female
- removed JP1, JP2: Jumper_NC_Small, Connector_PinHeader_2.54mm:PinHeader_1x02_P2.54mm_Vertical, symbol Device:Jumper_NC_Small
- removed U1: 4069, Package_DIP:DIP-14_W7.62mm, symbol 4xxx:4069
- added D1, D2: LED, LED_SMD:LED_0805_2012Metric_Pad1.15x1.40mm_HandSolder, symbol Device:LED
- added J1: FAN_PWR, Connector_JST:JST_XH_B2B-XH-A_1x02_P2.50mm_Vertical, symbol Connector:Conn_01x02_Female
- added J2: Conn_01x03_Female, Connector_JST:JST_XH_B3B-XH-A_1x03_P2.50mm_Vertical, symbol Connector:Conn_01x03_Female
- added J4: FAN_OUTPUT_2, Connector_JST:JST_XH_B4B-XH-A_1x04_P2.50mm_Vertical, symbol Connector:Conn_01x04_Female
- added J5: Conn_02x03_Odd_Even, Connector_PinHeader_2.54mm:PinHeader_2x03_P2.54mm_Vertical, symbol Connector_Generic:Conn_02x03_Odd_Even
- added R3, R4: R_US, Resistor_SMD:R_0805_2012Metric_Pad1.20x1.40mm_HandSolder, symbol Device:R_US
- J3: value IO -> FAN_OUTPUT_1
Connections:
- net CH2 is gone; now on net GND: J3.4 (Pin_4)
- net GND: now also J1.2 (Pin_2), J4.4 (Pin_4); no longer J3.2 (Pin_2)
- net IO_VCC: now also R1.2, J2.1 (Pin_1), J5.3 (Pin_3), J5.4 (Pin_4), R4.2; no longer J3.1 (Pin_1), R1.1, R2.1
- net PWM: now reaches R2.2
- net PWM: now also J3.2 (Pin_2), D1.1 (K), J2.3 (Pin_3), J4.2 (Pin_2)
- net CH1 renamed TAC
- net TAC: now also D2.1 (K), J2.2 (Pin_2), J4.3 (Pin_3), R3.2
- new net: J5.5 (Pin_5), R2.1
- new net: D1.2 (A), R1.1
- new net: J5.6 (Pin_6), R3.1
- new net: D2.2 (A), R4.1
- new net FAN_VCC: J1.1 (Pin_1), J3.1 (Pin_1), J4.1 (Pin_1)
- no-connect marks 0 -> 2
