File: tri-force-switch/wide-1515/bottom/bottom.kicad_pcb (KiCad board)
At the start: 4 copper layers, 50 x 26 mm, 7 parts, among them J1 Conn_01x02_Female, J2 Conn_01x02_Female, J3 BOLT_HOLE, J4 BOLT_HOLE, J5 BOLT_HOLE, J6 RING_HOLE, J7 BOLT_HOLE

Commit message: sync
Parts:
- J6: footprint custom-footprints:m4-d14-nut-outer-ring- -> custom-footprints:m3-d12-mounter-hole
Changed lines of the file:
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@@
     (pcbplotparams
       (layerselection 0x010fc_ffffffff)
-      (usegerberextensions false)
-      (usegerberattributes true)
-      (usegerberadvancedattributes true)
-      (creategerberjobfile true)
+      (usegerberextensions true)
+      (usegerberattributes false)
+      (usegerberadvancedattributes false)
+      (creategerberjobfile false)
       (excludeedgelayer true)
       (linewidth 0.100000)
@@
       (psa4output false)
       (plotreference true)
-      (plotvalue true)
+      (plotvalue false)
       (plotinvisibletext false)
       (padsonsilk false)
-      (subtractmaskfromsilk false)
+      (subtractmaskfromsilk true)
       (outputformat 1)
       (mirror false)
-      (drillshape 1)
+      (drillshape 0)
       (scaleselection 1)
-      (outputdirectory ""))
+      (outputdirectory "geber/"))
   )
   (net 0 "")
@@
       (net 2 "Net-(J1-Pad2)"))
   )
-  (module custom-footprints:m4-d14-nut-outer-ring- (layer F.Cu)
-    (at 80 90)
-    (fp_text reference J6 (at 0 0.5) (layer F.SilkS) hide
-      (effects (font (size 1 1) (thickness 0.15)))
-    )
-    (fp_text value RING_HOLE (at 0 -0.5) (layer F.Fab)
-      (effects (font (size 1 1) (thickness 0.15)))
-    )
-    (pad 1 thru_hole circle (at 0 0) (size 14 14) (drill 10) (layers *.Cu *.Mask)
-      (net 1 "Net-(J1-Pad1)"))
-  )
   (module custom-footprints:solder-pin-th-2pin (layer F.Cu)
     (at 59 101 270)
@@
       (net 2 "Net-(J1-Pad2)"))
   )
+  (module custom-footprints:m3-d12-mounter-hole (layer F.Cu)
+    (at 80 90)
+    (fp_text reference J6 (at 0 0.5) (layer F.SilkS)
+      (effects (font (size 1 1) (thickness 0.15)))
+    )
+    (fp_text value RING_HOLE (at 0 -0.5) (layer F.Fab)
+      (effects (font (size 1 1) (thickness 0.15)))
+    )
+    (pad 1 thru_hole circle (at 0 0) (size 12 12) (drill 9) (layers *.Cu *.Mask)
+      (net 1 "Net-(J1-Pad1)"))
+  )
   (gr_arc (start 103 84) (end 105 84) (angle -90) (layer Edge.Cuts) (width 0.05))
