File: tri-force-switch/wide-1515/bottom/bottom.sch (KiCad schematic (older format))
At the start: 7 parts, among them J1 Conn_01x02_Female, J2 Conn_01x02_Female, J3 BOLT_HOLE, J4 BOLT_HOLE, J5 BOLT_HOLE, J6 RING_HOLE, J7 BOLT_HOLE

Commit message: sync
Parts:
- J6: footprint custom-footprints:m4-d14-nut-outer-ring- -> custom-footprints:m3-d12-mounter-hole
Changed lines of the file:
@@
 F 0 "J6" H 3378 2326 50  0000 L CNN
 F 1 "RING_HOLE" H 3378 2235 50  0000 L CNN
-F 2 "custom-footprints:m4-d14-nut-outer-ring-" H 3350 2300 50  0001 C CNN
+F 2 "custom-footprints:m3-d12-mounter-hole" H 3350 2300 50  0001 C CNN
 F 3 "~" H 3350 2300 50  0001 C CNN
 	1    3350 2300
