File: tri-force-switch/wide-1515/top/top.kicad_pcb (KiCad board)
At the start: 4 copper layers, 50 x 26 mm, 5 parts, among them J1 BOLT_HOLE, J2 BOLT_HOLE, J3 BOLT_HOLE, J4 CENTER_BOLT, J5 BOLT_HOLE

Commit message: sync
Parts:
- J4: footprint custom-footprints:m4-d14-nut-mounter-hole -> custom-footprints:m3-d12-nut-mounter-hole
Changed lines of the file:
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@@
     (pcbplotparams
       (layerselection 0x010fc_ffffffff)
-      (usegerberextensions false)
-      (usegerberattributes true)
-      (usegerberadvancedattributes true)
-      (creategerberjobfile true)
+      (usegerberextensions true)
+      (usegerberattributes false)
+      (usegerberadvancedattributes false)
+      (creategerberjobfile false)
       (excludeedgelayer true)
       (linewidth 0.100000)
@@
       (psa4output false)
       (plotreference true)
-      (plotvalue true)
+      (plotvalue false)
       (plotinvisibletext false)
       (padsonsilk false)
-      (subtractmaskfromsilk false)
+      (subtractmaskfromsilk true)
       (outputformat 1)
       (mirror false)
-      (drillshape 1)
+      (drillshape 0)
       (scaleselection 1)
-      (outputdirectory ""))
+      (outputdirectory "geber/"))
   )
   (net 0 "")
@@
       (net 1 "Net-(J1-Pad1)"))
   )
-  (module custom-footprints:m4-d14-nut-mounter-hole (layer F.Cu)
-    (at 130 100)
-    (fp_text reference J4 (at 0 0.5) (layer F.SilkS) hide
-      (effects (font (size 1 1) (thickness 0.15)))
-    )
-    (fp_text value CENTER_BOLT (at 0 -0.5) (layer F.Fab)
-      (effects (font (size 1 1) (thickness 0.15)))
-    )
-    (pad 1 thru_hole circle (at 0 0) (size 14 14) (drill 4) (layers *.Cu *.Mask)
-      (net 1 "Net-(J1-Pad1)"))
-  )
   (module custom-footprints:m3-d8-mounting-hole (layer F.Cu)
     (at 143 113)
@@
       (net 1 "Net-(J1-Pad1)"))
   )
+  (module custom-footprints:m3-d12-nut-mounter-hole (layer F.Cu)
+    (at 130 100)
+    (fp_text reference J4 (at 0 0.5) (layer F.SilkS)
+      (effects (font (size 1 1) (thickness 0.15)))
+    )
+    (fp_text value CENTER_BOLT (at 0 -0.5) (layer F.Fab)
+      (effects (font (size 1 1) (thickness 0.15)))
+    )
+    (pad 1 thru_hole circle (at 0 0) (size 12 12) (drill 3) (layers *.Cu *.Mask)
+      (net 1 "Net-(J1-Pad1)"))
+  )
