File: tri-force-switch/wide-1515/top/top.sch (KiCad schematic (older format))
At the start: 5 parts, among them J1 BOLT_HOLE, J2 BOLT_HOLE, J3 BOLT_HOLE, J4 CENTER_BOLT, J5 BOLT_HOLE

Commit message: sync
Parts:
- J4: footprint custom-footprints:m4-d14-nut-mounter-hole -> custom-footprints:m3-d12-nut-mounter-hole
Changed lines of the file:
@@
 F 0 "J4" H 1778 2176 50  0000 L CNN
 F 1 "CENTER_BOLT" H 1778 2085 50  0000 L CNN
-F 2 "custom-footprints:m4-d14-nut-mounter-hole" H 1750 2150 50  0001 C CNN
+F 2 "custom-footprints:m3-d12-nut-mounter-hole" H 1750 2150 50  0001 C CNN
 F 3 "~" H 1750 2150 50  0001 C CNN
 	1    1750 2150
