File: pixel-battery-breakout/pixel-battery-breakout.sch (KiCad schematic (older format))
At the start: 7 parts, among them J1 BATT+, J2 BATT-, J3 GND_SHIELD, J4 Conn_01x02_Female, J5 Conn_01x04_Female

Commit message: sync
Parts:
- added J6, J7: TEST_POINT, custom-footprints:solder-pad, symbol Connector:Conn_01x01_Female
- JP1: value Jumper_NO_Small -> JP
Connections:
- net at J5.4 (Pin_4), JP1.2, R1.1: now also J7.1 (Pin_1)
- net at J3.1 (Pin_1), JP1.1, R1.2: now also J6.1 (Pin_1)
Changed lines of the file:
@@
 P 3950 2700
 F 0 "JP1" H 3950 2885 50  0000 C CNN
-F 1 "Jumper_NO_Small" H 3950 2600 50  0000 C CNN
+F 1 "JP" H 3950 2600 50  0000 C CNN
 F 2 "Jumper:SolderJumper-2_P1.3mm_Open_RoundedPad1.0x1.5mm" H 3950 2700 50  0001 C CNN
 F 3 "~" H 3950 2700 50  0001 C CNN
@@
 Wire Wire Line
 	4200 2000 4450 2000
+$Comp
+L Connector:Conn_01x01_Female J6
+U 1 1 63E2F8BB
+P 3800 3200
+F 0 "J6" H 3700 3300 50  0000 C CNN
+F 1 "TEST_POINT" H 4100 3200 50  0000 C CNN
+F 2 "custom-footprints:solder-pad" H 3800 3200 50  0001 C CNN
+F 3 "~" H 3800 3200 50  0001 C CNN
+	1    3800 3200
+	0    1    1    0
+$EndComp
+$Comp
+L Connector:Conn_01x01_Female J7
+U 1 1 63E31956
+P 4100 3200
+F 0 "J7" H 4000 3300 50  0000 C CNN
+F 1 "TEST_POINT" H 4350 3200 50  0000 C CNN
+F 2 "custom-footprints:solder-pad" H 4100 3200 50  0001 C CNN
+F 3 "~" H 4100 3200 50  0001 C CNN
+	1    4100 3200
+	0    1    1    0
+$EndComp
+Wire Wire Line
+	3800 2700 3800 3000
+Connection ~ 3800 2700
+Wire Wire Line
+	4100 3000 4100 2700
+Connection ~ 4100 2700
 $EndSCHEMATC
