File: audio-io-breakout-pajeromini/audio-io-breakout-pajeromini.kicad_pcb (KiCad board)
At the start: 2 copper layers, 30 x 22.5 mm, 12 parts, among them J1 TAPE, J2 Conn_01x04_Female

Commit message: sync2
Parts:
- added JP7: Jumper, Jumper:SolderJumper-2_P1.3mm_Open_RoundedPad1.0x1.5mm, B.Cu at (108.5, 82.7)
- moved JP1 1.50 mm to (103.0, 82.7)
- moved JP2 1.50 mm to (100.2, 82.7)
- moved JP3 1.50 mm to (92.0, 82.7)
- moved JP4 1.50 mm to (97.5, 82.7)
- moved JP5 1.50 mm to (94.8, 82.7)
- moved JP6 1.50 mm to (105.8, 82.7), turned to 90 degrees
Connections:
- JP1 pad 1: SG -> AG
- JP2 pad 1: SG -> AG
- JP6 pad 2: GND -> AG
Routing:
- net AG: track 0.00 -> 8.25 mm
- net SG: track 18.3 -> 11.6 mm
- net PWR-SW: track 3.01 -> 3.67 mm
- net NR: track 5.73 -> 6.35 mm
- net NL: track 5.82 -> 6.44 mm
Other:
- board text added: "AG-GND"
- board text added: "AG-SG"
- board text removed: "SG-GND"
