File: audio-io-breakout-pajeromini/audio-io-breakout-pajeromini.sch (KiCad schematic (older format))
At the start: 10 parts, among them J1 TAPE, J2 Conn_01x04_Female

Commit message: sync2
Parts:
- added JP7: Jumper, Jumper:SolderJumper-2_P1.3mm_Open_RoundedPad1.0x1.5mm, symbol Device:Jumper
Connections:
- net GND: now also JP7.1; no longer JP6.2
- net SG: no longer JP1.1, JP2.1
- new net AG: JP1.1, JP2.1, JP6.2, JP7.2
Changed lines of the file:
@@
 RL
 Text GLabel 1150 950  0    50   Input ~ 0
-SG
+AG
 Text GLabel 1150 1450 0    50   Input ~ 0
-SG
+AG
 Text GLabel 1150 2000 0    50   Input ~ 0
 PWR-SW
@@
 Text GLabel 1100 2950 0    50   Input ~ 0
 SG
-Text GLabel 1100 3050 0    50   Input ~ 0
+Text GLabel 1100 3200 0    50   Input ~ 0
 GND
 $Comp
@@
 Wire Wire Line
 	1100 2950 1300 2950
-Wire Wire Line
-	1900 3050 1900 2950
-Wire Wire Line
-	1100 3050 1900 3050
 Text GLabel 3900 4000 0    50   Input ~ 0
 MOTOR
@@
 	1    0    0    -1
 $EndComp
+Text GLabel 2350 2950 2    50   Input ~ 0
+AG
+$Comp
+L Device:Jumper JP7
+U 1 1 64092183
+P 1600 3200
+F 0 "JP7" H 1600 3464 50  0000 C CNN
+F 1 "Jumper" H 1600 3373 50  0000 C CNN
+F 2 "Jumper:SolderJumper-2_P1.3mm_Open_RoundedPad1.0x1.5mm" H 1600 3200 50  0001 C CNN
+F 3 "~" H 1600 3200 50  0001 C CNN
+	1    1600 3200
+	1    0    0    -1
+$EndComp
+Wire Wire Line
+	1100 3200 1300 3200
+Wire Wire Line
+	1900 2950 1900 3200
+Wire Wire Line
+	1900 2950 2350 2950
+Connection ~ 1900 2950
 $EndSCHEMATC
