File: tablet-usb-adapter/tablet-usb-adapter.kicad_pcb (KiCad board)
At the start: 2 copper layers, 50 x 20 mm, 12 parts, among them J1 PWR_SHIELD, J2 USB_HEADER, J3 USB_A, SW1 SW_Push

Commit message: sync
Other:
- board text added: "USB OTG Adapter"
Changed lines of the file:
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@@
-(kicad_pcb (version 20171130) (host pcbnew 5.1.9+dfsg1-1+deb11u1)
+(kicad_pcb (version 20171130) (host pcbnew 5.1.9+dfsg1-1)
   (general
     (thickness 1.6)
-    (drawings 45)
+    (drawings 46)
     (tracks 30)
     (zones 0)
@@
   )
   (setup
-    (last_trace_width 0.5)
+    (last_trace_width 0.25)
     (user_trace_width 0.5)
     (user_trace_width 1)
@@
     (pcbplotparams
       (layerselection 0x010fc_ffffffff)
-      (usegerberextensions false)
-      (usegerberattributes true)
-      (usegerberadvancedattributes true)
-      (creategerberjobfile true)
+      (usegerberextensions true)
+      (usegerberattributes false)
+      (usegerberadvancedattributes false)
+      (creategerberjobfile false)
       (excludeedgelayer true)
       (linewidth 0.100000)
@@
       (psa4output false)
       (plotreference true)
-      (plotvalue true)
+      (plotvalue false)
       (plotinvisibletext false)
       (padsonsilk false)
-      (subtractmaskfromsilk false)
+      (subtractmaskfromsilk true)
       (outputformat 1)
       (mirror false)
-      (drillshape 1)
+      (drillshape 0)
       (scaleselection 1)
-      (outputdirectory ""))
+      (outputdirectory "geber/"))
   )
   (net 0 "")
@@
       (effects (font (size 1 1) (thickness 0.15)))
     )
-    (fp_text user %R (at 0.3 0) (layer F.Fab)
-      (effects (font (size 1 1) (thickness 0.15)))
-    )
     (fp_circle (center 0 0) (end 2.8 0) (layer Cmts.User) (width 0.15))
     (fp_circle (center 0 0) (end 3.05 0) (layer F.CrtYd) (width 0.05))
+    (fp_text user %R (at 0.3 0) (layer F.Fab)
+      (effects (font (size 1 1) (thickness 0.15)))
+    )
     (pad 1 thru_hole circle (at 0 0) (size 5.6 5.6) (drill 3.2) (layers *.Cu *.Mask))
   )
@@
       (effects (font (size 1 1) (thickness 0.15)))
     )
-    (fp_text user %R (at 0.3 0) (layer F.Fab)
-      (effects (font (size 1 1) (thickness 0.15)))
-    )
     (fp_circle (center 0 0) (end 2.8 0) (layer Cmts.User) (width 0.15))
     (fp_circle (center 0 0) (end 3.05 0) (layer F.CrtYd) (width 0.05))
+    (fp_text user %R (at 0.3 0) (layer F.Fab)
+      (effects (font (size 1 1) (thickness 0.15)))
+    )
     (pad 1 thru_hole circle (at 0 0) (size 5.6 5.6) (drill 3.2) (layers *.Cu *.Mask))
   )
@@
       (effects (font (size 1 1) (thickness 0.15)))
     )
-    (fp_text user %R (at 0.3 0) (layer F.Fab)
-      (effects (font (size 1 1) (thickness 0.15)))
-    )
     (fp_circle (center 0 0) (end 2.8 0) (layer Cmts.User) (width 0.15))
     (fp_circle (center 0 0) (end 3.05 0) (layer F.CrtYd) (width 0.05))
+    (fp_text user %R (at 0.3 0) (layer F.Fab)
+      (effects (font (size 1 1) (thickness 0.15)))
+    )
     (pad 1 thru_hole circle (at 0 0) (size 5.6 5.6) (drill 3.2) (layers *.Cu *.Mask))
   )
@@
       (effects (font (size 1 1) (thickness 0.15)))
     )
-    (fp_text user %R (at 0.3 0) (layer F.Fab)
-      (effects (font (size 1 1) (thickness 0.15)))
-    )
     (fp_circle (center 0 0) (end 2.8 0) (layer Cmts.User) (width 0.15))
     (fp_circle (center 0 0) (end 3.05 0) (layer F.CrtYd) (width 0.05))
+    (fp_text user %R (at 0.3 0) (layer F.Fab)
+      (effects (font (size 1 1) (thickness 0.15)))
+    )
     (pad 1 thru_hole circle (at 0 0) (size 5.6 5.6) (drill 3.2) (layers *.Cu *.Mask))
   )
@@
       (effects (font (size 1 1) (thickness 0.15)))
     )
-    (fp_text user %R (at 0.3 0) (layer F.Fab)
-      (effects (font (size 1 1) (thickness 0.15)))
-    )
     (fp_circle (center 0 0) (end 2.8 0) (layer Cmts.User) (width 0.15))
     (fp_circle (center 0 0) (end 3.05 0) (layer F.CrtYd) (width 0.05))
+    (fp_text user %R (at 0.3 0) (layer F.Fab)
+      (effects (font (size 1 1) (thickness 0.15)))
+    )
     (pad 1 thru_hole circle (at 0 0) (size 5.6 5.6) (drill 3.2) (layers *.Cu *.Mask))
   )
@@
       (effects (font (size 0.5 0.5) (thickness 0.08)))
     )
-    (pad 1 smd roundrect (at -1 0) (size 1.2 1.4) (layers F.Cu F.Paste F.Mask) (roundrect_rratio 0.208333)
+    (pad 1 smd roundrect (at -1 0) (size 1.2 1.4) (layers F.Cu F.Paste F.Mask) (roundrect_rratio 0.2083325)
       (net 4 ID))
-    (pad 2 smd roundrect (at 1 0) (size 1.2 1.4) (layers F.Cu F.Paste F.Mask) (roundrect_rratio 0.208333)
+    (pad 2 smd roundrect (at 1 0) (size 1.2 1.4) (layers F.Cu F.Paste F.Mask) (roundrect_rratio 0.2083325)
       (net 3 SG))
     (model ${KISYS3DMOD}/Resistor_SMD.3dshapes/R_0805_2012Metric.wrl
@@
       (effects (font (size 0.5 0.5) (thickness 0.08)))
     )
-    (pad 1 smd roundrect (at -1 0 180) (size 1.2 1.4) (layers F.Cu F.Paste F.Mask) (roundrect_rratio 0.208333)
+    (pad 1 smd roundrect (at -1 0 180) (size 1.2 1.4) (layers F.Cu F.Paste F.Mask) (roundrect_rratio 0.2083325)
       (net 4 ID))
-    (pad 2 smd roundrect (at 1 0 180) (size 1.2 1.4) (layers F.Cu F.Paste F.Mask) (roundrect_rratio 0.208333)
+    (pad 2 smd roundrect (at 1 0 180) (size 1.2 1.4) (layers F.Cu F.Paste F.Mask) (roundrect_rratio 0.2083325)
       (net 7 V+))
     (model ${KISYS3DMOD}/Resistor_SMD.3dshapes/R_0805_2012Metric.wrl
@@
     )
   )
+  (gr_text "USB OTG\nAdapter" (at 140.716 106.934) (layer F.SilkS)
+    (effects (font (size 1 1) (thickness 0.15)) (justify left))
+  )
   (gr_line (start 133 104) (end 133 117.5) (layer Dwgs.User) (width 0.15))
   (gr_line (start 141.75 104) (end 133 104) (layer Dwgs.User) (width 0.15))
   (gr_line (start 124.25 104) (end 141.75 104) (layer Dwgs.User) (width 0.15))
-  (gr_text Rev.1 (at 144.5 107.5) (layer F.SilkS)
+  (gr_text Rev.1 (at 145.542 109.474) (layer F.SilkS)
     (effects (font (size 1 1) (thickness 0.15)))
   )

Commit message: sync
Parts:
- removed GND-ID: Jumper_NO_Small, Jumper:SolderJumper-2_P1.3mm_Open_RoundedPad1.0x1.5mm
- added G***: juice-plus_logo_3k, custom-footprints:juice-plus_logo_3k, B.Cu at (132.5, 110.5)
- moved R2 3.50 mm to (144.5, 118.0)
- moved R1 1.50 mm to (144.5, 120.0)
Routing:
- net ID: track 21.8 -> 15.8 mm, vias 0 -> 1
- net SG: track 4.10 -> 0.00 mm
- net V+: track 14.8 -> 12.6 mm, vias 0 -> 1

Commit message: sync2
Parts:
- added JP1: Jumper_NO_Small, Jumper:SolderJumper-2_P1.3mm_Open_RoundedPad1.0x1.5mm, F.Cu at (144.4, 114.0)
Connections:
- J2 pad 2: SG -> V-
- J3 pad 4: SG -> V-
- R1 pad 2: SG -> V-
Routing:
- net SG: track 0.00 -> 25.1 mm
- added copper zone on B.Cu, net V-
- added copper zone on F.Cu, net V-
- removed copper zone on B.Cu, net SG
- removed copper zone on F.Cu, net SG
Other:
- board text added: "Rev.1b"
- board text added: "S-G"
- board text removed: "Rev.1"
