File: zenfone-max-m2-ext/tablet-usb-adapter/tablet-usb-adapter.kicad_pcb (KiCad board)
At the start: 2 copper layers, 51.5 x 27.5 mm, 19 parts, among them J1 MINI-USB, J2 COMBO_CONN, J3 USB_A, K1 OMRON_G6L, Q1 NCV8402, U1 ATtiny85-20PU

Commit message: sync
Parts:
- removed the G*** at (111.5, 74.5)
- removed the G*** at (125.0, 76.5)
- added J4: bridge, Connector_PinSocket_1.27mm:PinSocket_1x01_P1.27mm_Vertical, F.Cu at (108.2, 75.5)
- added J5: bridge, Connector_PinSocket_1.27mm:PinSocket_1x01_P1.27mm_Vertical, F.Cu at (110.2, 71.0)
- added J6: bridge, Connector_PinSocket_1.27mm:PinSocket_1x01_P1.27mm_Vertical, F.Cu at (108.2, 71.0)
- added J7: bridge, Connector_PinSocket_1.27mm:PinSocket_1x01_P1.27mm_Vertical, F.Cu at (110.2, 75.5)
- added S1: Switch, custom-footprints:switch-side-btn, F.Cu at (109.2, 64.3)
- added U2: R3111-SOT235, Package_TO_SOT_SMD:SOT-23-5, B.Cu at (118.5, 76.5)
- moved G*** 25.0 mm to (138.0, 75.8)
- moved JP1 11.0 mm to (113.7, 77.2), turned to 0 degrees
Routing:
- net GND: track 25.2 -> 0.50 mm, vias 0 -> 5
- net Net-(U1-Pad1): track 0.00 -> 20.7 mm, vias 0 -> 1
- net TABLET_SHIELD: track 18.4 -> 25.6 mm
- net Net-(J6-Pad1): track 0.00 -> 4.87 mm
- net Net-(J5-Pad1): track 0.00 -> 4.87 mm
- net VCC: track 68.9 -> 72.9 mm, vias 1 -> 0
Other:
- board text added: "Bridge shield"
- board text added: "Rev.2e"
- board text removed: "Rev.2c"
