File: zenfone-max-m2-ext/tablet-usb-adapter/tablet-usb-adapter.sch (KiCad schematic (older format))
At the start: 11 parts, among them J1 MINI-USB, J2 COMBO_CONN, J3 USB_A, K1 OMRON_G6L, Q1 NCV8402, U1 ATtiny85-20PU

Commit message: sync
Parts:
- added J4, J5, J6, J7: bridge, Connector_PinSocket_1.27mm:PinSocket_1x01_P1.27mm_Vertical, symbol Connector:Conn_01x01_Female
- added S1: Switch, custom-footprints:switch-side-btn, symbol custom-symbols:Switch
- added U2: R3111-SOT235, Package_TO_SOT_SMD:SOT-23-5, symbol custom-symbols:R3111-SOT235
Connections:
- net GND: now also U2.3 (GND)
- net TABLET_GND: now also J7.1 (Pin_1)
- net TABLET_SHIELD: now also J4.1 (Pin_1)
- net VCC: now also U2.2 (VCC)
- net at U1.1 (~RESET~/PB5): now also U2.1 (OUT)
- new net: J5.1 (Pin_1), S1.1
- new net: J6.1 (Pin_1), S1.2
- no-connect marks 6 -> 9
Changed lines of the file:
@@
 Wire Wire Line
 	6250 3700 6250 4000
-Wire Wire Line
-	6250 4450 6250 4300
 $Comp
 L Device:R_US R1
@@
 Wire Wire Line
 	4800 4550 4800 4300
-NoConn ~ 5400 3900
 NoConn ~ 5400 3800
 NoConn ~ 5400 3500
@@
 Text GLabel 3500 2000 0    50   Input ~ 0
 TABLET_SHIELD
+$Comp
+L custom-symbols:Switch S1
+U 1 1 64C59169
+P 4675 5600
+F 0 "S1" H 4675 5925 50  0000 C CNN
+F 1 "Switch" H 4675 5834 50  0000 C CNN
+F 2 "custom-footprints:switch-side-btn" H 4675 5600 50  0001 C CNN
+F 3 "" H 4675 5600 50  0001 C CNN
+	1    4675 5600
+	1    0    0    -1
+$EndComp
+Text GLabel 5525 4750 0    50   Input ~ 0
+GND
+Text GLabel 5525 4625 0    50   Input ~ 0
+VCC
+NoConn ~ 6100 4500
+NoConn ~ 6100 4750
+$Comp
+L custom-symbols:R3111-SOT235 U2
+U 1 1 64C79BCE
+P 5850 4625
+F 0 "U2" H 5812 4975 50  0000 C CNN
+F 1 "R3111-SOT235" H 5812 4884 50  0000 C CNN
+F 2 "Package_TO_SOT_SMD:SOT-23-5" H 5850 4625 50  0001 C CNN
+F 3 "" H 5850 4625 50  0001 C CNN
+	1    5850 4625
+	1    0    0    -1
+$EndComp
+Text GLabel 3825 5500 0    50   Input ~ 0
+TABLET_SHIELD
+Wire Wire Line
+	6250 4300 6250 4450
+Wire Wire Line
+	5525 4500 5525 3900
+Wire Wire Line
+	5525 3900 5400 3900
+$Comp
+L Connector:Conn_01x01_Female J4
+U 1 1 64CA18E4
+P 4025 5500
+F 0 "J4" H 4053 5526 50  0000 L CNN
+F 1 "bridge" H 4000 5650 50  0000 L CNN
+F 2 "Connector_PinSocket_1.27mm:PinSocket_1x01_P1.27mm_Vertical" H 4025 5500 50  0001 C CNN
+F 3 "~" H 4025 5500 50  0001 C CNN
+	1    4025 5500
+	1    0    0    -1
+$EndComp
+$Comp
+L Connector:Conn_01x01_Female J5
+U 1 1 64CA42A2
+P 4300 5500
+F 0 "J5" H 4192 5275 50  0000 C CNN
+F 1 "bridge" H 4192 5366 50  0000 C CNN
+F 2 "Connector_PinSocket_1.27mm:PinSocket_1x01_P1.27mm_Vertical" H 4300 5500 50  0001 C CNN
+F 3 "~" H 4300 5500 50  0001 C CNN
+	1    4300 5500
+	-1   0    0    1
+$EndComp
+$Comp
+L Connector:Conn_01x01_Female J6
+U 1 1 64CAE55E
+P 5050 5500
+F 0 "J6" H 5078 5526 50  0000 L CNN
+F 1 "bridge" H 5025 5650 50  0000 L CNN
+F 2 "Connector_PinSocket_1.27mm:PinSocket_1x01_P1.27mm_Vertical" H 5050 5500 50  0001 C CNN
+F 3 "~" H 5050 5500 50  0001 C CNN
+	1    5050 5500
+	1    0    0    -1
+$EndComp
+$Comp
+L Connector:Conn_01x01_Female J7
+U 1 1 64CAF139
+P 5275 5500
+F 0 "J7" H 5303 5526 50  0000 L CNN
+F 1 "bridge" H 5250 5650 50  0000 L CNN
+F 2 "Connector_PinSocket_1.27mm:PinSocket_1x01_P1.27mm_Vertical" H 5275 5500 50  0001 C CNN
+F 3 "~" H 5275 5500 50  0001 C CNN
+	1    5275 5500
+	-1   0    0    1
+$EndComp
+Text GLabel 5475 5500 2    50   Input ~ 0
+TABLET_GND
+NoConn ~ 4500 5675
+NoConn ~ 4850 5675
 $EndSCHEMATC
